File: iconcard/iconcard.kicad_sch (KiCad schematic)
At the start: 30 parts, among them J1 JST-SH, J2 PinSocket 2.54mm, J3 JST-PH, J4 USB_C_Receptacle_PowerOnly_6P, U1 STM32G030F6Px, U2 KXTJ3-1057, U3 MCP73831-2-OT, U4 AP2112K-3.3

Commit message: Update tact switch to SKRPACE010, fix LCSC part numbers, add production files
Co-Authored-By: Claude Opus 4.6 <noreply@anthropic.com>
Parts:
- BOOT1, RST1: footprint RST/BOOT (タクトSW):KEY-SMD_4P-L6.0-W6.0-P4.50-LS10.0 -> SKRPACE010:KEY-SMD_4P-L4.2-W3.2-P2.20-LS4.6; LCSC (none) -> C139797
- C1, C3, C4, C7: LCSC (none) -> C309458
- C2: LCSC (none) -> C19666
- C5, C6, C8, C9: LCSC (none) -> C380332
- CHG1: renamed from CHARGE_STATUS1; LCSC (none) -> C2286
- J1: LCSC (none) -> C7527619
- J2: now not fitted; now left out of the parts list
- J3: LCSC (none) -> C968533
- J4: LCSC (none) -> C456012
- Power1: LCSC (none) -> C49023767
- R1: LCSC (none) -> C25744
- R2, R8: LCSC (none) -> C4109
- R3, R4: LCSC (none) -> C25879
- R5, R6: LCSC (none) -> C25905
- R7: LCSC (none) -> C25903
- STAT1: renamed from STM32_STATUS1; LCSC (none) -> C12624
- U1: LCSC (none) -> C724040
- U2: LCSC (none) -> C442603
- U3: LCSC (none) -> C424093
- U4: LCSC (none) -> C51118

Commit message: Move STAT LED from PA6 to PA8, update R2 to 4.7K
Co-Authored-By: Claude Opus 4.6 (1M context) <noreply@anthropic.com>
Parts:
- R2: value 2K -> 4.7K
Connections:
- net at U1.13 (PA6): no longer R2.2
- net at U1.15 (PA8/PB0/PB1/PB2): now also R2.2
Changed lines of the file:
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@@
 	)
 	(no_connect
-		(at 180.34 76.2)
+		(at 231.14 86.36)
 	)
 	(no_connect
-		(at 231.14 91.44)
+		(at 180.34 76.2)
 	)
 	(no_connect
@@
 	(wire
 		(pts
-			(xy 245.11 64.77) (xy 245.11 86.36)
+			(xy 245.11 64.77) (xy 245.11 91.44)
 		)
 		(stroke
@@
 	(wire
 		(pts
+			(xy 245.11 91.44) (xy 231.14 91.44)
+		)
+		(stroke
+			(width 0)
+			(type default)
+		)
+	)
+	(wire
+		(pts
 			(xy 236.22 78.74) (xy 236.22 41.91)
 		)
@@
 	(wire
 		(pts
-			(xy 245.11 86.36) (xy 231.14 86.36)
-		)
-		(stroke
-			(width 0)
-			(type default)
-		)
-	)
-	(wire
-		(pts
 			(xy 173.99 153.67) (xy 151.13 153.67)
 		)
@@
 			)
 		)
-		(property "Value" "2K"
+		(property "Value" "4.7K"
 			(at 247.65 62.2299 0)
 			(effects

Commit message: Add BL MOSFET driver, SWD test points, update J2 to 8-pin
Co-Authored-By: Claude Opus 4.6 (1M context) <noreply@anthropic.com>
Parts:
- removed J2: PinSocket 2.54mm, Connector_PinSocket_2.54mm:PinSocket_1x07_P2.54mm_Vertical, symbol Connector:Conn_01x07_Socket
- added J2: Conn_01x08_Socket, Connector_PinSocket_2.54mm:PinSocket_1x08_P2.54mm_Vertical, symbol Connector:Conn_01x08_Socket
- added Q1: 2N7002, Package_TO_SOT_SMD:SOT-23, symbol Transistor_FET:2N7002
- added R10: 100K, Resistor_SMD:R_0402_1005Metric, symbol Device:R
- added R9: 100, Resistor_SMD:R_0402_1005Metric, symbol Device:R
- added TP1: SWDIO, TestPoint:TestPoint_THTPad_D1.0mm_Drill0.5mm, symbol Connector:TestPoint
- added TP2: SWCLK, TestPoint:TestPoint_THTPad_D1.0mm_Drill0.5mm, symbol Connector:TestPoint
- added TP3: GND, TestPoint:TestPoint_THTPad_D1.0mm_Drill0.5mm, symbol Connector:TestPoint
- R2: LCSC C4109 -> C25900
Connections:
- net CS: now also J2.7 (Pin_7)
- net DC: now also J2.6 (Pin_6)
- net GND: now also J2.1 (Pin_1), Q1.2 (S), R10.2, TP3.1
- net PA2_TX: now also J2.5 (Pin_5)
- net SCL: now also J2.3 (Pin_3)
- net SDA: now also J2.4 (Pin_4)
- net VCC: now also J2.2 (Pin_2)
- net at R2.2, U1.15 (PA8/PB0/PB1/PB2): now also R10.1, R9.1
- net SWDIO: now reaches U1.18 (PA13)
- net SWDIO: now also TP1.1
- net at BOOT1.1, R1.1, U1.19 (PA14/PA15): now also TP2.1
- new net: Q1.1 (G), R9.2
- new net BL: J2.8 (Pin_8), Q1.3 (D)
- no-connect marks 7 -> 6
Other:
- moved on the sheet: J1
