File: puchi_pix/puchi_pix.kicad_pcb (KiCad board)
At the start: 2 copper layers, 35 x 30.5 mm, 38 parts, among them J1 JST-SH, J2 Conn_01x08_Socket, J3 JST-PH, J4 USB_C_Receptacle_PowerOnly_6P, Q1 2N7002, U1 STM32G030F6Px, U2 KXTJ3-1057, U3 MCP73831-2-OT, U4 AP2112K-3.3

Commit message: Add pixel art logo to PCB silkscreen
Co-Authored-By: Claude Opus 4.6 (1M context) <noreply@anthropic.com>
Parts:
- added ?: , brand:puchi_pix_logo, F.Cu at (49.0, 37.0)
Other:
- board text added: "Puchi-Pix by @yacchin1205, Mizunashi-Lab"
- board text added: "V0.9"
- board text removed: "by Mizunashi-Lab @yacchin1205"
