File: puchi_pix/puchi_pix.kicad_pcb (KiCad board)
At the start: 2 copper layers, 35 x 30.5 mm, 39 parts, among them J1 JST-SH, J2 Conn_01x08_Socket, J3 JST-PH, J4 USB_C_Receptacle_PowerOnly_6P, Q1 2N7002, U1 STM32G030F6Px, U2 KXTJ3-1057, U3 MCP73831-2-OT, U4 AP2112K-3.3

Commit message: Add files for JLCPCB
Other:
- board text added: "SWCLK"
- board text added: "SWDIO"
Changed lines of the file:
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@@
 			(at 0 2 0)
 			(layer "B.SilkS")
+			(hide yes)
 			(effects
 				(font
@@
 			(at -0.5 2 0)
 			(layer "B.SilkS")
+			(hide yes)
 			(effects
 				(font
@@
 			(at 2.5 0 0)
 			(layer "B.SilkS")
+			(hide yes)
 			(effects
 				(font
@@
 		)
 	)
+	(gr_text "GND"
+		(at 26 25.5 0)
+		(layer "B.SilkS")
+		(effects
+			(font
+				(size 0.8 0.8)
+				(thickness 0.1)
+			)
+			(justify left bottom mirror)
+		)
+	)
+	(gr_text "SWDIO"
+		(at 38 25.5 0)
+		(layer "B.SilkS")
+		(effects
+			(font
+				(size 0.8 0.8)
+				(thickness 0.1)
+			)
+			(justify left bottom mirror)
+		)
+	)
 	(gr_text "DC"
 		(at 24.5 31.5 0)
@@
 	)
 	(gr_text "BL"
-		(at 24.5 26.5 0)
+		(at 24.5 27 0)
 		(layer "B.SilkS")
 		(effects
@@
 		(layer "B.SilkS")
 		(effects
+			(font
+				(size 0.8 0.8)
+				(thickness 0.1)
+			)
+			(justify left bottom mirror)
+		)
+	)
+	(gr_text "SWCLK"
+		(at 52 25.5 0)
+		(layer "B.SilkS")
+		(effects
