File: puchi_pix/puchi_pix.kicad_pcb (KiCad board)
At the start: 2 copper layers, 35 x 30.5 mm, 39 parts, among them J1 JST-SH, J2 Conn_01x08_Socket, J3 JST-PH, J4 USB_C_Receptacle_PowerOnly_6P, Q1 2N7002, U1 STM32G030F6Px, U2 KXTJ3-1057, U3 MCP73831-2-OT, U4 AP2112K-3.3

Commit message: Finalize puchi_pix/esp32 layout and regenerate JLCPCB production files (puchi_pix V0_95)
Co-Authored-By: Claude Opus 4.8 (1M context) <noreply@anthropic.com>
Parts:
- J2: moved to B.Cu
- moved REF** 24.0 mm to (22.0, 25.0)
- moved J2 14.8 mm to (21.5, 29.2)
- moved TP3 10.5 mm to (34.0, 23.5)
- moved R2 1.00 mm to (34.0, 28.0)
- moved STAT1 0.66 mm to (35.5, 25.7)
- moved R8 0.50 mm to (25.0, 38.5), turned to -90 degrees
Routing:
- net /BL: track 24.1 -> 45.7 mm
- net /SCL: track 14.1 -> 21.1 mm, vias 0 -> 2
- net /CS: track 8.93 -> 15.5 mm, vias 0 -> 2
- net /DC: track 7.77 -> 11.9 mm, vias 0 -> 2
- net /PA2_TX: track 18.7 -> 21.5 mm, vias 0 -> 2
- net Net-(U3-STAT): track 14.9 -> 12.2 mm
- net /PA3_RX: track 14.5 -> 16.8 mm
- net GND: track 29.4 -> 28.2 mm
- net Net-(U1-PA8/PB0/PB1/PB2): track 12.1 -> 11.1 mm
- net /VCC: track 76.9 -> 76.3 mm, vias 2 -> 4
Other:
- board text added: "V0.95"
- board text removed: "V0.9"
