File: puchi_pix_esp32/puchi_pix_esp32.kicad_sch (KiCad schematic)
At the start: 38 parts, among them J1 USB_C_Receptacle_USB2.0_16P, J2 Conn_01x08, J3 JST-PH, J4 Conn_01x04_Socket, SW1 BOOT, SW2 RST, U1 ESP32-C3-MINI-1, U2 MCP73831-2-OT, U3 KXTJ3-1057, U4 AP2112K-3.3

Commit message: Update D1 to green LED (C12624) with R3=4.7k and add production files
Co-Authored-By: Claude Opus 4.6 (1M context) <noreply@anthropic.com>
Parts:
- D1: LCSC C72041 -> C12624
- R3: value 39 -> 4.7k; LCSC C25110 -> C25900
Changed lines of the file:
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@@
 			)
 		)
-		(property "LCSC" "C72041"
+		(property "LCSC" "C12624"
 			(at 20.32 121.92 90)
 			(effects
@@
 			)
 		)
-		(property "Value" "39"
+		(property "Value" "4.7k"
 			(at 22.86 113.0299 0)
 			(effects
@@
 			)
 		)
-		(property "LCSC" "C25110"
+		(property "LCSC" "C25900"
 			(at 20.32 111.76 0)
 			(effects

Commit message: Finalize puchi_pix/esp32 layout and regenerate JLCPCB production files (puchi_pix V0_95)
Co-Authored-By: Claude Opus 4.8 (1M context) <noreply@anthropic.com>
Parts:
- removed J2: Conn_01x08, Connector_JST:JST_PH_S8B-PH-SM4-TB_1x08-1MP_P2.00mm_Horizontal, symbol Connector_Generic:Conn_01x08
- added J2: Conn_01x08_Socket, Connector_PinSocket_2.00mm:PinSocket_1x08_P2.00mm_Vertical, symbol Connector:Conn_01x08_Socket
Connections:
- net +3.3V: now also J2.8 (Pin_8)
- net BL: now also J2.1 (Pin_1)
- net CLK: now also J2.5 (Pin_5)
- net CS: now also J2.4 (Pin_4)
- net DC: now also J2.3 (Pin_3)
- net DIN: now also J2.6 (Pin_6)
- net GND: now also J2.7 (Pin_7)
- net RST: now also J2.2 (Pin_2)
Changed lines of the file:
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@@
 	)
 	(symbol
+		(lib_id "Connector:Conn_01x08_Socket")
+		(at 212.09 135.89 0)
+		(mirror x)
+		(unit 1)
+		(exclude_from_sim no)
+		(in_bom no)
+		(on_board yes)
+		(dnp no)
+		(property "Reference" "J2"
+			(at 213.868 122.936 0)
+			(effects
+				(font
+					(size 1.27 1.27)
+				)
+			)
+		)
+		(property "Value" "Conn_01x08_Socket"
+			(at 213.106 146.05 0)
+			(effects
+				(font
+					(size 1.27 1.27)
+				)
+			)
+		)
+		(property "Footprint" "Connector_PinSocket_2.00mm:PinSocket_1x08_P2.00mm_Vertical"
+			(at 212.09 135.89 0)
+			(effects
+				(font
+					(size 1.27 1.27)
+				)
+				(hide yes)
+			)
+		)
+		(property "Datasheet" "~"
+			(at 212.09 135.89 0)
+			(effects
+				(font
+					(size 1.27 1.27)
+				)
+				(hide yes)
+			)
+		)
+		(property "Description" "Generic connector, single row, 01x08, script generated"
+			(at 212.09 135.89 0)
+			(effects
+				(font
+					(size 1.27 1.27)
+				)
+				(hide yes)
+			)
+		)
+		(pin "8"
+		)
+		(pin "6"
+		)
+		(pin "5"
+		)
+		(pin "3"
+		)
+		(pin "7"
+		)
+		(pin "4"
+		)
+		(pin "2"
+		)
+		(pin "1"
+		)
+		(instances
+			(project ""
+				(path "/3c749848-9eab-418d-8f91-4e5f63c41477"
+					(reference "J2")
+					(unit 1)
+				)
+			)
+		)
+	)
+	(symbol
 		(lib_id "Device:C")
 		(at 231.14 107.95 0)
@@
 					(unit 1)
 				)
-			)
-		)
-	)
-	(symbol
-		(lib_id "Connector_Generic:Conn_01x08")
-		(at 212.09 135.89 0)
-		(mirror x)
-		(unit 1)
-		(exclude_from_sim no)
-		(in_bom yes)
-		(on_board yes)
-		(dnp no)
-		(property "Reference" "J2"
-			(at 214.63 135.8901 0)
-			(effects
-				(font
-					(size 1.27 1.27)
-				)
-				(justify left)
-			)
-		)
-		(property "Value" "Conn_01x08"
-			(at 214.63 133.3501 0)
-			(effects
-				(font
-					(size 1.27 1.27)
-				)
-				(justify left)
-			)
-		)
-		(property "Footprint" "Connector_JST:JST_PH_S8B-PH-SM4-TB_1x08-1MP_P2.00mm_Horizontal"
-			(at 212.09 135.89 0)
-			(effects
-				(font
-					(size 1.27 1.27)
-				)
-				(hide yes)
-			)
-		)
-		(property "Datasheet" "~"
-			(at 212.09 135.89 0)
-			(effects
-				(font
-					(size 1.27 1.27)
-				)
-				(hide yes)
-			)
-		)
-		(property "Description" "Generic connector, single row, 01x08, script generated (kicad-library-utils/schlib/autogen/connector/)"
-			(at 212.09 135.89 0)
-			(effects
-				(font
-					(size 1.27 1.27)
-				)
-				(hide yes)
-			)
-		)
-		(property "LCSC" "C265121"
-			(at 212.09 135.89 0)
-			(effects
-				(font
-					(size 1.27 1.27)
-				)
-				(hide yes)
-			)
-		)
-		(pin "1"
-		)
-		(pin "2"
-		)
-		(pin "5"
-		)
-		(pin "4"
-		)
-		(pin "3"
-		)
-		(pin "6"
-		)
-		(pin "7"
-		)
-		(pin "8"
-		)
-		(instances
-			(project "puchi_pix_esp32"
-				(path "/3c749848-9eab-418d-8f91-4e5f63c41477"
-					(reference "J2")
-					(unit 1)
-				)
