File: hardware/puchi_pix_card/display.kicad_sch (KiCad schematic)
At the start: 0 parts

Commit message: Add the display sheet: 16x16 FM-B2020RGBA matrix, MBI5153 x3, 74HCT595 + PFET row scan
Co-Authored-By: Claude Fable 5 <noreply@anthropic.com>
Parts:
- added C101, C102, C103, C104, C105: 100nF, Capacitor_SMD:C_0402_1005Metric, symbol Device:C
- added D101, D102, D103, D104, D105, D106, D107, D108, D109, D110, D111, D112, D113, D114, D115, D116, D117, D118, D119, D120, D121, D122, D123, D124, D125, D126, D127, D128, D129, D130, D131, D132, D133, D134, D135, D136, D137, D138, D139, D140, D141, D142, D143, D144, D145, D146, D147, D148, D149, D150, D151, D152, D153, D154, D155, D156, D157, D158, D159, D160, D161, D162, D163, D164, D165, D166, D167, D168, D169, D170, D171, D172, D173, D174, D175, D176, D177, D178, D179, D180, D181, D182, D183, D184, D185, D186, D187, D188, D189, D190, D191, D192, D193, D194, D195, D196, D197, D198, D199, D200, D201, D202, D203, D204, D205, D206, D207, D208, D209, D210, D211, D212, D213, D214, D215, D216, D217, D218, D219, D220, D221, D222, D223, D224, D225, D226, D227, D228, D229, D230, D231, D232, D233, D234, D235, D236, D237, D238, D239, D240, D241, D242, D243, D244, D245, D246, D247, D248, D249, D250, D251, D252, D253, D254, D255, D256, D257, D258, D259, D260, D261, D262, D263, D264, D265, D266, D267, D268, D269, D270, D271, D272, D273, D274, D275, D276, D277, D278, D279, D280, D281, D282, D283, D284, D285, D286, D287, D288, D289, D290, D291, D292, D293, D294, D295, D296, D297, D298, D299, D300, D301, D302, D303, D304, D305, D306, D307, D308, D309, D310, D311, D312, D313, D314, D315, D316, D317, D318, D319, D320, D321, D322, D323, D324, D325, D326, D327, D328, D329, D330, D331, D332, D333, D334, D335, D336, D337, D338, D339, D340, D341, D342, D343, D344, D345, D346, D347, D348, D349, D350, D351, D352, D353, D354, D355, D356: FM-B2020RGBA-HG, puchi_pix_card:LED_FM-B2020RGBA, symbol puchi_pix_card:FM-B2020RGBA
- added Q101, Q102, Q103, Q104, Q105, Q106, Q107, Q108, Q109, Q110, Q111, Q112, Q113, Q114, Q115, Q116: AO3401A, Package_TO_SOT_SMD:SOT-23, symbol Transistor_FET:AO3401A
- added R101: 1.5k, Resistor_SMD:R_0402_1005Metric, symbol Device:R
- added R102: 2.4k, Resistor_SMD:R_0402_1005Metric, symbol Device:R
- added R103: 4.7k, Resistor_SMD:R_0402_1005Metric, symbol Device:R
- added R104: 10k, Resistor_SMD:R_0402_1005Metric, symbol Device:R
- added U101: MBI5153GP (R), puchi_pix_card:SSOP24L-150-0.64, symbol puchi_pix_card:MBI5153GP
- added U102: MBI5153GP (G), puchi_pix_card:SSOP24L-150-0.64, symbol puchi_pix_card:MBI5153GP
- added U103: MBI5153GP (B), puchi_pix_card:SSOP24L-150-0.64, symbol puchi_pix_card:MBI5153GP
- added U104, U105: 74HCT595, Package_SO:SOIC-16_3.9x9.9mm_P1.27mm, symbol 74xx:74HCT595
Connections:
- new net: R101.1, U101.23 (R-EXT)
- new net: R102.1, U102.23 (R-EXT)
- new net: R103.1, U103.23 (R-EXT)
- new net: U104.9 (QH'), U105.14 (SER)
- new net: U101.22 (SDO), U102.2 (SDI)
- new net: U102.22 (SDO), U103.2 (SDI)
- new net +3V3P: C101.1, C102.1, C103.1, U101.24 (VDD), U102.24 (VDD), U103.24 (VDD)
- new net +5V: C104.1, C105.1, Q101.2 (S), Q102.2 (S), Q103.2 (S), Q104.2 (S), Q105.2 (S), Q106.2 (S), Q107.2 (S), Q108.2 (S), Q109.2 (S), Q110.2 (S), Q111.2 (S), Q112.2 (S), Q113.2 (S), Q114.2 (S), Q115.2 (S), Q116.2 (S), R104.1, U104.10 (~{SRCLR}), U104.16 (VCC), U105.10 (~{SRCLR}), U105.16 (VCC)
- new net COL_B0: D101.2 (BK), D117.2 (BK), D133.2 (BK), D149.2 (BK), D165.2 (BK), D181.2 (BK), D197.2 (BK), D213.2 (BK), D229.2 (BK), D245.2 (BK), D261.2 (BK), D277.2 (BK), D293.2 (BK), D309.2 (BK), D325.2 (BK), D341.2 (BK), U103.5 (OUT0)
- new net COL_B1: D102.2 (BK), D118.2 (BK), D134.2 (BK), D150.2 (BK), D166.2 (BK), D182.2 (BK), D198.2 (BK), D214.2 (BK), D230.2 (BK), D246.2 (BK), D262.2 (BK), D278.2 (BK), D294.2 (BK), D310.2 (BK), D326.2 (BK), D342.2 (BK), U103.6 (OUT1)
- new net COL_B10: D111.2 (BK), D127.2 (BK), D143.2 (BK), D159.2 (BK), D175.2 (BK), D191.2 (BK), D207.2 (BK), D223.2 (BK), D239.2 (BK), D255.2 (BK), D271.2 (BK), D287.2 (BK), D303.2 (BK), D319.2 (BK), D335.2 (BK), D351.2 (BK), U103.15 (OUT10)
- new net COL_B11: D112.2 (BK), D128.2 (BK), D144.2 (BK), D160.2 (BK), D176.2 (BK), D192.2 (BK), D208.2 (BK), D224.2 (BK), D240.2 (BK), D256.2 (BK), D272.2 (BK), D288.2 (BK), D304.2 (BK), D320.2 (BK), D336.2 (BK), D352.2 (BK), U103.16 (OUT11)
- new net COL_B12: D113.2 (BK), D129.2 (BK), D145.2 (BK), D161.2 (BK), D177.2 (BK), D193.2 (BK), D209.2 (BK), D225.2 (BK), D241.2 (BK), D257.2 (BK), D273.2 (BK), D289.2 (BK), D305.2 (BK), D321.2 (BK), D337.2 (BK), D353.2 (BK), U103.17 (OUT12)
- new net COL_B13: D114.2 (BK), D130.2 (BK), D146.2 (BK), D162.2 (BK), D178.2 (BK), D194.2 (BK), D210.2 (BK), D226.2 (BK), D242.2 (BK), D258.2 (BK), D274.2 (BK), D290.2 (BK), D306.2 (BK), D322.2 (BK), D338.2 (BK), D354.2 (BK), U103.18 (OUT13)
- new net COL_B14: D115.2 (BK), D131.2 (BK), D147.2 (BK), D163.2 (BK), D179.2 (BK), D195.2 (BK), D211.2 (BK), D227.2 (BK), D243.2 (BK), D259.2 (BK), D275.2 (BK), D291.2 (BK), D307.2 (BK), D323.2 (BK), D339.2 (BK), D355.2 (BK), U103.19 (OUT14)
- new net COL_B15: D116.2 (BK), D132.2 (BK), D148.2 (BK), D164.2 (BK), D180.2 (BK), D196.2 (BK), D212.2 (BK), D228.2 (BK), D244.2 (BK), D260.2 (BK), D276.2 (BK), D292.2 (BK), D308.2 (BK), D324.2 (BK), D340.2 (BK), D356.2 (BK), U103.20 (OUT15)
- new net COL_B2: D103.2 (BK), D119.2 (BK), D135.2 (BK), D151.2 (BK), D167.2 (BK), D183.2 (BK), D199.2 (BK), D215.2 (BK), D231.2 (BK), D247.2 (BK), D263.2 (BK), D279.2 (BK), D295.2 (BK), D311.2 (BK), D327.2 (BK), D343.2 (BK), U103.7 (OUT2)
- new net COL_B3: D104.2 (BK), D120.2 (BK), D136.2 (BK), D152.2 (BK), D168.2 (BK), D184.2 (BK), D200.2 (BK), D216.2 (BK), D232.2 (BK), D248.2 (BK), D264.2 (BK), D280.2 (BK), D296.2 (BK), D312.2 (BK), D328.2 (BK), D344.2 (BK), U103.8 (OUT3)
- new net COL_B4: D105.2 (BK), D121.2 (BK), D137.2 (BK), D153.2 (BK), D169.2 (BK), D185.2 (BK), D201.2 (BK), D217.2 (BK), D233.2 (BK), D249.2 (BK), D265.2 (BK), D281.2 (BK), D297.2 (BK), D313.2 (BK), D329.2 (BK), D345.2 (BK), U103.9 (OUT4)
- new net COL_B5: D106.2 (BK), D122.2 (BK), D138.2 (BK), D154.2 (BK), D170.2 (BK), D186.2 (BK), D202.2 (BK), D218.2 (BK), D234.2 (BK), D250.2 (BK), D266.2 (BK), D282.2 (BK), D298.2 (BK), D314.2 (BK), D330.2 (BK), D346.2 (BK), U103.10 (OUT5)
- new net COL_B6: D107.2 (BK), D123.2 (BK), D139.2 (BK), D155.2 (BK), D171.2 (BK), D187.2 (BK), D203.2 (BK), D219.2 (BK), D235.2 (BK), D251.2 (BK), D267.2 (BK), D283.2 (BK), D299.2 (BK), D315.2 (BK), D331.2 (BK), D347.2 (BK), U103.11 (OUT6)
- new net COL_B7: D108.2 (BK), D124.2 (BK), D140.2 (BK), D156.2 (BK), D172.2 (BK), D188.2 (BK), D204.2 (BK), D220.2 (BK), D236.2 (BK), D252.2 (BK), D268.2 (BK), D284.2 (BK), D300.2 (BK), D316.2 (BK), D332.2 (BK), D348.2 (BK), U103.12 (OUT7)
- new net COL_B8: D109.2 (BK), D125.2 (BK), D141.2 (BK), D157.2 (BK), D173.2 (BK), D189.2 (BK), D205.2 (BK), D221.2 (BK), D237.2 (BK), D253.2 (BK), D269.2 (BK), D285.2 (BK), D301.2 (BK), D317.2 (BK), D333.2 (BK), D349.2 (BK), U103.13 (OUT8)
- new net COL_B9: D110.2 (BK), D126.2 (BK), D142.2 (BK), D158.2 (BK), D174.2 (BK), D190.2 (BK), D206.2 (BK), D222.2 (BK), D238.2 (BK), D254.2 (BK), D270.2 (BK), D286.2 (BK), D302.2 (BK), D318.2 (BK), D334.2 (BK), D350.2 (BK), U103.14 (OUT9)
- new net COL_G0: D101.4 (GK), D117.4 (GK), D133.4 (GK), D149.4 (GK), D165.4 (GK), D181.4 (GK), D197.4 (GK), D213.4 (GK), D229.4 (GK), D245.4 (GK), D261.4 (GK), D277.4 (GK), D293.4 (GK), D309.4 (GK), D325.4 (GK), D341.4 (GK), U102.5 (OUT0)
- new net COL_G1: D102.4 (GK), D118.4 (GK), D134.4 (GK), D150.4 (GK), D166.4 (GK), D182.4 (GK), D198.4 (GK), D214.4 (GK), D230.4 (GK), D246.4 (GK), D262.4 (GK), D278.4 (GK), D294.4 (GK), D310.4 (GK), D326.4 (GK), D342.4 (GK), U102.6 (OUT1)
- new net COL_G10: D111.4 (GK), D127.4 (GK), D143.4 (GK), D159.4 (GK), D175.4 (GK), D191.4 (GK), D207.4 (GK), D223.4 (GK), D239.4 (GK), D255.4 (GK), D271.4 (GK), D287.4 (GK), D303.4 (GK), D319.4 (GK), D335.4 (GK), D351.4 (GK), U102.15 (OUT10)
- new net COL_G11: D112.4 (GK), D128.4 (GK), D144.4 (GK), D160.4 (GK), D176.4 (GK), D192.4 (GK), D208.4 (GK), D224.4 (GK), D240.4 (GK), D256.4 (GK), D272.4 (GK), D288.4 (GK), D304.4 (GK), D320.4 (GK), D336.4 (GK), D352.4 (GK), U102.16 (OUT11)
- new net COL_G12: D113.4 (GK), D129.4 (GK), D145.4 (GK), D161.4 (GK), D177.4 (GK), D193.4 (GK), D209.4 (GK), D225.4 (GK), D241.4 (GK), D257.4 (GK), D273.4 (GK), D289.4 (GK), D305.4 (GK), D321.4 (GK), D337.4 (GK), D353.4 (GK), U102.17 (OUT12)
- new net COL_G13: D114.4 (GK), D130.4 (GK), D146.4 (GK), D162.4 (GK), D178.4 (GK), D194.4 (GK), D210.4 (GK), D226.4 (GK), D242.4 (GK), D258.4 (GK), D274.4 (GK), D290.4 (GK), D306.4 (GK), D322.4 (GK), D338.4 (GK), D354.4 (GK), U102.18 (OUT13)
- new net COL_G14: D115.4 (GK), D131.4 (GK), D147.4 (GK), D163.4 (GK), D179.4 (GK), D195.4 (GK), D211.4 (GK), D227.4 (GK), D243.4 (GK), D259.4 (GK), D275.4 (GK), D291.4 (GK), D307.4 (GK), D323.4 (GK), D339.4 (GK), D355.4 (GK), U102.19 (OUT14)
- new net COL_G15: D116.4 (GK), D132.4 (GK), D148.4 (GK), D164.4 (GK), D180.4 (GK), D196.4 (GK), D212.4 (GK), D228.4 (GK), D244.4 (GK), D260.4 (GK), D276.4 (GK), D292.4 (GK), D308.4 (GK), D324.4 (GK), D340.4 (GK), D356.4 (GK), U102.20 (OUT15)
- new net COL_G2: D103.4 (GK), D119.4 (GK), D135.4 (GK), D151.4 (GK), D167.4 (GK), D183.4 (GK), D199.4 (GK), D215.4 (GK), D231.4 (GK), D247.4 (GK), D263.4 (GK), D279.4 (GK), D295.4 (GK), D311.4 (GK), D327.4 (GK), D343.4 (GK), U102.7 (OUT2)
- new net COL_G3: D104.4 (GK), D120.4 (GK), D136.4 (GK), D152.4 (GK), D168.4 (GK), D184.4 (GK), D200.4 (GK), D216.4 (GK), D232.4 (GK), D248.4 (GK), D264.4 (GK), D280.4 (GK), D296.4 (GK), D312.4 (GK), D328.4 (GK), D344.4 (GK), U102.8 (OUT3)
- new net COL_G4: D105.4 (GK), D121.4 (GK), D137.4 (GK), D153.4 (GK), D169.4 (GK), D185.4 (GK), D201.4 (GK), D217.4 (GK), D233.4 (GK), D249.4 (GK), D265.4 (GK), D281.4 (GK), D297.4 (GK), D313.4 (GK), D329.4 (GK), D345.4 (GK), U102.9 (OUT4)
- new net COL_G5: D106.4 (GK), D122.4 (GK), D138.4 (GK), D154.4 (GK), D170.4 (GK), D186.4 (GK), D202.4 (GK), D218.4 (GK), D234.4 (GK), D250.4 (GK), D266.4 (GK), D282.4 (GK), D298.4 (GK), D314.4 (GK), D330.4 (GK), D346.4 (GK), U102.10 (OUT5)
- new net COL_G6: D107.4 (GK), D123.4 (GK), D139.4 (GK), D155.4 (GK), D171.4 (GK), D187.4 (GK), D203.4 (GK), D219.4 (GK), D235.4 (GK), D251.4 (GK), D267.4 (GK), D283.4 (GK), D299.4 (GK), D315.4 (GK), D331.4 (GK), D347.4 (GK), U102.11 (OUT6)
- new net COL_G7: D108.4 (GK), D124.4 (GK), D140.4 (GK), D156.4 (GK), D172.4 (GK), D188.4 (GK), D204.4 (GK), D220.4 (GK), D236.4 (GK), D252.4 (GK), D268.4 (GK), D284.4 (GK), D300.4 (GK), D316.4 (GK), D332.4 (GK), D348.4 (GK), U102.12 (OUT7)
- new net COL_G8: D109.4 (GK), D125.4 (GK), D141.4 (GK), D157.4 (GK), D173.4 (GK), D189.4 (GK), D205.4 (GK), D221.4 (GK), D237.4 (GK), D253.4 (GK), D269.4 (GK), D285.4 (GK), D301.4 (GK), D317.4 (GK), D333.4 (GK), D349.4 (GK), U102.13 (OUT8)
- new net COL_G9: D110.4 (GK), D126.4 (GK), D142.4 (GK), D158.4 (GK), D174.4 (GK), D190.4 (GK), D206.4 (GK), D222.4 (GK), D238.4 (GK), D254.4 (GK), D270.4 (GK), D286.4 (GK), D302.4 (GK), D318.4 (GK), D334.4 (GK), D350.4 (GK), U102.14 (OUT9)
- new net COL_R0: D101.1 (RK), D117.1 (RK), D133.1 (RK), D149.1 (RK), D165.1 (RK), D181.1 (RK), D197.1 (RK), D213.1 (RK), D229.1 (RK), D245.1 (RK), D261.1 (RK), D277.1 (RK), D293.1 (RK), D309.1 (RK), D325.1 (RK), D341.1 (RK), U101.5 (OUT0)
- new net COL_R1: D102.1 (RK), D118.1 (RK), D134.1 (RK), D150.1 (RK), D166.1 (RK), D182.1 (RK), D198.1 (RK), D214.1 (RK), D230.1 (RK), D246.1 (RK), D262.1 (RK), D278.1 (RK), D294.1 (RK), D310.1 (RK), D326.1 (RK), D342.1 (RK), U101.6 (OUT1)
- new net COL_R10: D111.1 (RK), D127.1 (RK), D143.1 (RK), D159.1 (RK), D175.1 (RK), D191.1 (RK), D207.1 (RK), D223.1 (RK), D239.1 (RK), D255.1 (RK), D271.1 (RK), D287.1 (RK), D303.1 (RK), D319.1 (RK), D335.1 (RK), D351.1 (RK), U101.15 (OUT10)
- new net COL_R11: D112.1 (RK), D128.1 (RK), D144.1 (RK), D160.1 (RK), D176.1 (RK), D192.1 (RK), D208.1 (RK), D224.1 (RK), D240.1 (RK), D256.1 (RK), D272.1 (RK), D288.1 (RK), D304.1 (RK), D320.1 (RK), D336.1 (RK), D352.1 (RK), U101.16 (OUT11)
- new net COL_R12: D113.1 (RK), D129.1 (RK), D145.1 (RK), D161.1 (RK), D177.1 (RK), D193.1 (RK), D209.1 (RK), D225.1 (RK), D241.1 (RK), D257.1 (RK), D273.1 (RK), D289.1 (RK), D305.1 (RK), D321.1 (RK), D337.1 (RK), D353.1 (RK), U101.17 (OUT12)
- new net COL_R13: D114.1 (RK), D130.1 (RK), D146.1 (RK), D162.1 (RK), D178.1 (RK), D194.1 (RK), D210.1 (RK), D226.1 (RK), D242.1 (RK), D258.1 (RK), D274.1 (RK), D290.1 (RK), D306.1 (RK), D322.1 (RK), D338.1 (RK), D354.1 (RK), U101.18 (OUT13)
- new net COL_R14: D115.1 (RK), D131.1 (RK), D147.1 (RK), D163.1 (RK), D179.1 (RK), D195.1 (RK), D211.1 (RK), D227.1 (RK), D243.1 (RK), D259.1 (RK), D275.1 (RK), D291.1 (RK), D307.1 (RK), D323.1 (RK), D339.1 (RK), D355.1 (RK), U101.19 (OUT14)
- new net COL_R15: D116.1 (RK), D132.1 (RK), D148.1 (RK), D164.1 (RK), D180.1 (RK), D196.1 (RK), D212.1 (RK), D228.1 (RK), D244.1 (RK), D260.1 (RK), D276.1 (RK), D292.1 (RK), D308.1 (RK), D324.1 (RK), D340.1 (RK), D356.1 (RK), U101.20 (OUT15)
- new net COL_R2: D103.1 (RK), D119.1 (RK), D135.1 (RK), D151.1 (RK), D167.1 (RK), D183.1 (RK), D199.1 (RK), D215.1 (RK), D231.1 (RK), D247.1 (RK), D263.1 (RK), D279.1 (RK), D295.1 (RK), D311.1 (RK), D327.1 (RK), D343.1 (RK), U101.7 (OUT2)
- new net COL_R3: D104.1 (RK), D120.1 (RK), D136.1 (RK), D152.1 (RK), D168.1 (RK), D184.1 (RK), D200.1 (RK), D216.1 (RK), D232.1 (RK), D248.1 (RK), D264.1 (RK), D280.1 (RK), D296.1 (RK), D312.1 (RK), D328.1 (RK), D344.1 (RK), U101.8 (OUT3)
- new net COL_R4: D105.1 (RK), D121.1 (RK), D137.1 (RK), D153.1 (RK), D169.1 (RK), D185.1 (RK), D201.1 (RK), D217.1 (RK), D233.1 (RK), D249.1 (RK), D265.1 (RK), D281.1 (RK), D297.1 (RK), D313.1 (RK), D329.1 (RK), D345.1 (RK), U101.9 (OUT4)
- new net COL_R5: D106.1 (RK), D122.1 (RK), D138.1 (RK), D154.1 (RK), D170.1 (RK), D186.1 (RK), D202.1 (RK), D218.1 (RK), D234.1 (RK), D250.1 (RK), D266.1 (RK), D282.1 (RK), D298.1 (RK), D314.1 (RK), D330.1 (RK), D346.1 (RK), U101.10 (OUT5)
- new net COL_R6: D107.1 (RK), D123.1 (RK), D139.1 (RK), D155.1 (RK), D171.1 (RK), D187.1 (RK), D203.1 (RK), D219.1 (RK), D235.1 (RK), D251.1 (RK), D267.1 (RK), D283.1 (RK), D299.1 (RK), D315.1 (RK), D331.1 (RK), D347.1 (RK), U101.11 (OUT6)
- new net COL_R7: D108.1 (RK), D124.1 (RK), D140.1 (RK), D156.1 (RK), D172.1 (RK), D188.1 (RK), D204.1 (RK), D220.1 (RK), D236.1 (RK), D252.1 (RK), D268.1 (RK), D284.1 (RK), D300.1 (RK), D316.1 (RK), D332.1 (RK), D348.1 (RK), U101.12 (OUT7)
- new net COL_R8: D109.1 (RK), D125.1 (RK), D141.1 (RK), D157.1 (RK), D173.1 (RK), D189.1 (RK), D205.1 (RK), D221.1 (RK), D237.1 (RK), D253.1 (RK), D269.1 (RK), D285.1 (RK), D301.1 (RK), D317.1 (RK), D333.1 (RK), D349.1 (RK), U101.13 (OUT8)
- new net COL_R9: D110.1 (RK), D126.1 (RK), D142.1 (RK), D158.1 (RK), D174.1 (RK), D190.1 (RK), D206.1 (RK), D222.1 (RK), D238.1 (RK), D254.1 (RK), D270.1 (RK), D286.1 (RK), D302.1 (RK), D318.1 (RK), D334.1 (RK), D350.1 (RK), U101.14 (OUT9)
- new net GCLK: U101.21 (GCLK), U102.21 (GCLK), U103.21 (GCLK)
- new net GND: C101.2, C102.2, C103.2, C104.2, C105.2, R101.2, R102.2, R103.2, U101.1 (GND), U102.1 (GND), U103.1 (GND), U104.8 (GND), U105.8 (GND)
- new net MBI_DCLK: U101.3 (DCLK), U102.3 (DCLK), U103.3 (DCLK)
- new net MBI_LE: U101.4 (LE), U102.4 (LE), U103.4 (LE)
- new net MBI_SDI: U101.2 (SDI)
- new net MBI_SDO: U103.22 (SDO)
- new net ROW0: D101.3 (A), D102.3 (A), D103.3 (A), D104.3 (A), D105.3 (A), D106.3 (A), D107.3 (A), D108.3 (A), D109.3 (A), D110.3 (A), D111.3 (A), D112.3 (A), D113.3 (A), D114.3 (A), D115.3 (A), D116.3 (A), Q101.3 (D)
- new net ROW1: D117.3 (A), D118.3 (A), D119.3 (A), D120.3 (A), D121.3 (A), D122.3 (A), D123.3 (A), D124.3 (A), D125.3 (A), D126.3 (A), D127.3 (A), D128.3 (A), D129.3 (A), D130.3 (A), D131.3 (A), D132.3 (A), Q102.3 (D)
- new net ROW10: D261.3 (A), D262.3 (A), D263.3 (A), D264.3 (A), D265.3 (A), D266.3 (A), D267.3 (A), D268.3 (A), D269.3 (A), D270.3 (A), D271.3 (A), D272.3 (A), D273.3 (A), D274.3 (A), D275.3 (A), D276.3 (A), Q111.3 (D)
- new net ROW11: D277.3 (A), D278.3 (A), D279.3 (A), D280.3 (A), D281.3 (A), D282.3 (A), D283.3 (A), D284.3 (A), D285.3 (A), D286.3 (A), D287.3 (A), D288.3 (A), D289.3 (A), D290.3 (A), D291.3 (A), D292.3 (A), Q112.3 (D)
- new net ROW12: D293.3 (A), D294.3 (A), D295.3 (A), D296.3 (A), D297.3 (A), D298.3 (A), D299.3 (A), D300.3 (A), D301.3 (A), D302.3 (A), D303.3 (A), D304.3 (A), D305.3 (A), D306.3 (A), D307.3 (A), D308.3 (A), Q113.3 (D)
- new net ROW13: D309.3 (A), D310.3 (A), D311.3 (A), D312.3 (A), D313.3 (A), D314.3 (A), D315.3 (A), D316.3 (A), D317.3 (A), D318.3 (A), D319.3 (A), D320.3 (A), D321.3 (A), D322.3 (A), D323.3 (A), D324.3 (A), Q114.3 (D)
- new net ROW14: D325.3 (A), D326.3 (A), D327.3 (A), D328.3 (A), D329.3 (A), D330.3 (A), D331.3 (A), D332.3 (A), D333.3 (A), D334.3 (A), D335.3 (A), D336.3 (A), D337.3 (A), D338.3 (A), D339.3 (A), D340.3 (A), Q115.3 (D)
- new net ROW15: D341.3 (A), D342.3 (A), D343.3 (A), D344.3 (A), D345.3 (A), D346.3 (A), D347.3 (A), D348.3 (A), D349.3 (A), D350.3 (A), D351.3 (A), D352.3 (A), D353.3 (A), D354.3 (A), D355.3 (A), D356.3 (A), Q116.3 (D)
- new net ROW2: D133.3 (A), D134.3 (A), D135.3 (A), D136.3 (A), D137.3 (A), D138.3 (A), D139.3 (A), D140.3 (A), D141.3 (A), D142.3 (A), D143.3 (A), D144.3 (A), D145.3 (A), D146.3 (A), D147.3 (A), D148.3 (A), Q103.3 (D)
- new net ROW3: D149.3 (A), D150.3 (A), D151.3 (A), D152.3 (A), D153.3 (A), D154.3 (A), D155.3 (A), D156.3 (A), D157.3 (A), D158.3 (A), D159.3 (A), D160.3 (A), D161.3 (A), D162.3 (A), D163.3 (A), D164.3 (A), Q104.3 (D)
- new net ROW4: D165.3 (A), D166.3 (A), D167.3 (A), D168.3 (A), D169.3 (A), D170.3 (A), D171.3 (A), D172.3 (A), D173.3 (A), D174.3 (A), D175.3 (A), D176.3 (A), D177.3 (A), D178.3 (A), D179.3 (A), D180.3 (A), Q105.3 (D)
- new net ROW5: D181.3 (A), D182.3 (A), D183.3 (A), D184.3 (A), D185.3 (A), D186.3 (A), D187.3 (A), D188.3 (A), D189.3 (A), D190.3 (A), D191.3 (A), D192.3 (A), D193.3 (A), D194.3 (A), D195.3 (A), D196.3 (A), Q106.3 (D)
- new net ROW6: D197.3 (A), D198.3 (A), D199.3 (A), D200.3 (A), D201.3 (A), D202.3 (A), D203.3 (A), D204.3 (A), D205.3 (A), D206.3 (A), D207.3 (A), D208.3 (A), D209.3 (A), D210.3 (A), D211.3 (A), D212.3 (A), Q107.3 (D)
- new net ROW7: D213.3 (A), D214.3 (A), D215.3 (A), D216.3 (A), D217.3 (A), D218.3 (A), D219.3 (A), D220.3 (A), D221.3 (A), D222.3 (A), D223.3 (A), D224.3 (A), D225.3 (A), D226.3 (A), D227.3 (A), D228.3 (A), Q108.3 (D)
- new net ROW8: D229.3 (A), D230.3 (A), D231.3 (A), D232.3 (A), D233.3 (A), D234.3 (A), D235.3 (A), D236.3 (A), D237.3 (A), D238.3 (A), D239.3 (A), D240.3 (A), D241.3 (A), D242.3 (A), D243.3 (A), D244.3 (A), Q109.3 (D)
- new net ROW9: D245.3 (A), D246.3 (A), D247.3 (A), D248.3 (A), D249.3 (A), D250.3 (A), D251.3 (A), D252.3 (A), D253.3 (A), D254.3 (A), D255.3 (A), D256.3 (A), D257.3 (A), D258.3 (A), D259.3 (A), D260.3 (A), Q110.3 (D)
- new net SR_NOE: R104.2, U104.13 (~{OE}), U105.13 (~{OE})
- new net SR_Q0: Q101.1 (G), U104.15 (QA)
- new net SR_Q1: Q102.1 (G), U104.1 (QB)
- new net SR_Q10: Q111.1 (G), U105.2 (QC)
- new net SR_Q11: Q112.1 (G), U105.3 (QD)
- new net SR_Q12: Q113.1 (G), U105.4 (QE)
- new net SR_Q13: Q114.1 (G), U105.5 (QF)
- new net SR_Q14: Q115.1 (G), U105.6 (QG)
- new net SR_Q15: Q116.1 (G), U105.7 (QH)
- new net SR_Q2: Q103.1 (G), U104.2 (QC)
- new net SR_Q3: Q104.1 (G), U104.3 (QD)
- new net SR_Q4: Q105.1 (G), U104.4 (QE)
- new net SR_Q5: Q106.1 (G), U104.5 (QF)
- new net SR_Q6: Q107.1 (G), U104.6 (QG)
- new net SR_Q7: Q108.1 (G), U104.7 (QH)
- new net SR_Q8: Q109.1 (G), U105.15 (QA)
- new net SR_Q9: Q110.1 (G), U105.1 (QB)
- new net SR_RCLK: U104.12 (RCLK), U105.12 (RCLK)
- new net SR_SER: U104.14 (SER)
- new net SR_SRCLK: U104.11 (SRCLK), U105.11 (SRCLK)
- no-connect marks 0 -> 1
Other:
- note added: "Columns: COL_R/G/B c = cathode buses (COL0 left) -> MBI5153 OUT c. Chain MCU SDI -> U101(R) -> U102(G) -> U103(B) -> MCU SDO."
- note added: "Rext: IOUT=(0.61V/Rext)x24 (MBI5153 p21) -> R 1.5k=9.8mA, G 2.4k=6.1mA, B 4.7k=3.1mA max; config gain 12.5-200%."
- note added: "Scan: ROW r = anode bus (ROW0 top), driven by Q1xx (AO3401A high side from +5V) via 74HCT595 SR_Q r."
